Commit message: Add grand finale capstone: mission control and real-world chapter
- Add Part 23 grand finale docs and demo cheatsheet
- Add CatchMission action, mission_control and mission_client nodes
- Add grand_finale launch file and config
- Wire up interfaces, setup.py, and spider_bot urdf updates

Co-Authored-By: Claude Opus 4.8 <noreply@anthropic.com>

File: src/spider_bot/urdf/spider_bot.urdf.xacro (robot description, xacro)
@@ -35,5 +35,7 @@
   <xacro:property name="mount_x" value="0.12"/>
   <xacro:property name="mount_y" value="0.08"/>
-  <xacro:property name="pi" value="3.14159265359"/>
+  <!-- xacro already provides pi as a built-in constant in ${} expressions,
+       so there is no property to declare here. Defining our own would trigger
+       "redefining global symbol: pi", which the launch file treats as fatal. -->
   <!-- ============================================================= -->
   <!-- Materials (colours in RViz).                                   -->
